Commit message: FEAT : File Upload

File: hyrian_description/urdf/gazebo_control.xacro (robot description, xacro)
@@ -15,5 +15,5 @@
             <robot_base_frame>base_link</robot_base_frame>
             <publish_odom>true</publish_odom>
-            <publish_odom_tf>true</publish_odom_tf>
+            <publish_odom_tf>false</publish_odom_tf>
             <publish_wheel_tf>true</publish_wheel_tf>
         </plugin>

File: hyrian_description/urdf/hyrian.xacro (robot description, xacro)
@@ -22,4 +22,11 @@
   </collision>
 </link>
+  <!-- footprint 추가 -->
+<link name="base_footprint"/>
+<joint name="base_joint" type="fixed">
+  <parent link="base_link"/>
+  <child link="base_footprint" />
+  <origin xyz="0 0.0 0.0" rpy="0 0 0.0"/>
+</joint>
 <link name="caster_1">
   <inertial>
@@ -42,24 +49,4 @@
   </collision>
 </link>
-<!-- <link name="lidar_1">
-  <inertial>
-    <origin xyz="2.5778920109686965e-09 6.0217946361192236e-18 0.023813967631461597" rpy="0 0 0"/>
-    <mass value="1.482019447760714"/>
-    <inertia ixx="0.000761" iyy="0.000761" izz="0.000958" ixy="0.0" iyz="0.0" ixz="0.0"/>
-  </inertial>
-  <visual>
-    <origin xyz="-0.068 0.0 -0.049" rpy="0 0 0"/>
-    <geometry>
-      <mesh filename="file://$(find hyrian_description)/meshes/lidar_1.stl" scale="0.001 0.001 0.001"/>
-    </geometry>
-    <material name="silver"/>
-  </visual>
-  <collision>
-    <origin xyz="-0.068 0.0 -0.049" rpy="0 0 0"/>
-    <geometry>
-      <mesh filename="file://$(find hyrian_description)/meshes/lidar_1.stl" scale="0.001 0.001 0.001"/>
-    </geometry>
-  </collision>
-</link> -->
 <link name="right_wheel_1">
   <inertial>
@@ -102,14 +89,9 @@
   </collision>
 </link>
-<joint name="��ü 15" type="fixed">
+<joint name="caster_joint" type="fixed">
   <origin xyz="-0.279 0.0 0.043" rpy="0 0 0"/>
   <parent link="base_link"/>
   <child link="caster_1"/>
 </joint>
-<!-- <joint name="��ü 13" type="fixed">
-  <origin xyz="0.068 0.0 0.049" rpy="0 0 0"/>
-  <parent link="base_link"/>
-  <child link="lidar_1"/>
-</joint> -->
 <joint name="right_wheel_joint" type="continuous">
   <origin xyz="0.0 -0.2118 0.0" rpy="0 0 0"/>
@@ -124,4 +106,5 @@
   <axis xyz="-0.0 1.0 -0.0"/>
 </joint>
+<!--
 <gazebo reference="base_link">
   <material>Gazebo/White</material>
@@ -137,13 +120,7 @@
   <self_collide>true</self_collide>
 </gazebo>
-<!-- <gazebo reference="lidar_1">
+<gazebo reference="caster_1">
   <material>Gazebo/White</material>
   <self_collide>true</self_collide>
 </gazebo> -->
-<gazebo reference="caster_1">
-  <material>Gazebo/White</material>
-  <mu1>0.001</mu1>
-  <mu2>0.001</mu2>
-  <self_collide>true</self_collide>
-</gazebo>
 </robot>

File: hyrian_description/urdf/robot.urdf.xacro (robot description, xacro)
@@ -9,5 +9,4 @@
     </xacro:unless>
     <xacro:include filename="hyrian.xacro" />
-    <xacro:include filename="lidar.xacro" />
-    <!-- <xacro:include filename="camera.xacro" /> -->
+    <xacro:include filename="sensor.xacro" />
 </robot>
